Commit message: Pnp updated to work with sawyer_irl_project!

File: robotiq_2f_85_gripper_visualization/urdf/robotiq_arg2f_85_model_macro.xacro (robot description, xacro)
@@ -74,4 +74,5 @@
     </link>
   </xacro:macro>
+<mass value="0.00853198276973456" />
   <xacro:macro name="inner_finger" params="prefix fingerprefix stroke">
     <link name="${prefix}${fingerprefix}_inner_finger">
