Commit message: Alter the color of the gripper so a blob finder can detect it

File: robotiq_2f_85_gripper_visualization/urdf/robotiq_arg2f.xacro (robot description, xacro)
@@ -13,7 +13,5 @@
           <mesh filename="package://robotiq_2f_85_gripper_visualization/meshes/visual/robotiq_arg2f_85_base_link.dae" scale="0.001 0.001 0.001"/>
         </geometry>
-        <material name="">
-          <color rgba="0.1 0.1 0.1 1" />
-        </material>
+        <material name="blue"/>
       </visual>
       <collision>

File: robotiq_2f_85_gripper_visualization/urdf/robotiq_arg2f_85_model.xacro (robot description, xacro)
@@ -1,4 +1,7 @@
 <?xml version="1.0"?>
 <robot name="robotiq_arg2f_85_model" xmlns:xacro="http://www.ros.org/wiki/xacro">
+  <material name="blue">
+	<color rgba="0 0 0.8 1"/>
+  </material>
   <xacro:include filename="$(find robotiq_2f_85_gripper_visualization)/urdf/robotiq_arg2f_85_model_macro.xacro" />
   <xacro:include filename="$(find robotiq_2f_85_gripper_visualization)/urdf/gazebo.urdf.xacro"/>

File: robotiq_2f_85_gripper_visualization/urdf/robotiq_arg2f_85_model_macro.xacro (robot description, xacro)
@@ -14,7 +14,5 @@
           <mesh filename="package://robotiq_2f_85_gripper_visualization/meshes/visual/robotiq_arg2f_85_outer_knuckle.dae" scale="0.001 0.001 0.001"/>
         </geometry>
-        <material name="">
-          <color rgba="0.792156862745098 0.819607843137255 0.933333333333333 1" />
-        </material>
+        <material name="blue"/>
       </visual>
       <collision>
@@ -38,7 +36,5 @@
           <mesh filename="package://robotiq_2f_85_gripper_visualization/meshes/visual/robotiq_arg2f_85_outer_finger.dae" scale="0.001 0.001 0.001"/>
         </geometry>
-        <material name="">
-          <color rgba="0.1 0.1 0.1 1" />
-        </material>
+        <material name="blue"/>
       </visual>
       <collision>
@@ -62,7 +58,5 @@
           <mesh filename="package://robotiq_2f_85_gripper_visualization/meshes/visual/robotiq_arg2f_85_inner_knuckle.dae" scale="0.001 0.001 0.001"/>
         </geometry>
-        <material name="">
-          <color rgba="0.1 0.1 0.1 1" />
-        </material>
+        <material name="blue"/>
       </visual>
       <collision>
@@ -87,7 +81,5 @@
           <mesh filename="package://robotiq_2f_85_gripper_visualization/meshes/visual/robotiq_arg2f_85_inner_finger.dae" scale="0.001 0.001 0.001"/>
         </geometry>
-        <material name="">
-          <color rgba="0.1 0.1 0.1 1" />
-        </material>
+        <material name="blue"/>
       </visual>
       <collision>
@@ -107,7 +99,5 @@
           <box size="0.022 0.00635 0.0375"/>
         </geometry>
-        <material name="">
-          <color rgba="0.9 0.9 0.9 1" />
-        </material>
+        <material name="blue"/>
       </visual>
       <collision>
@@ -151,7 +141,5 @@
           <cylinder length="0.02" radius="0.0025"/>
         </geometry>
-        <material name="">
-          <color rgba="0.1 0.1 0.1 1" />
-        </material>
+        <material name="blue"/>
       </visual>
       <collision>
